File: bottom/mysterium-bottom.kicad_pcb (KiCad board)
At the start: 2 copper layers, 347.7 x 146.6 mm, 22 parts

Commit message: Mysterium Iso additions
Parts:
- moved REF** 1.50 mm to (79.4, 178.6)
Changed lines of the file:
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@@
     (pcbplotparams
       (layerselection 0x010f0_ffffffff)
-      (usegerberextensions false)
+      (usegerberextensions true)
       (usegerberattributes false)
       (usegerberadvancedattributes false)
       (creategerberjobfile false)
-      (excludeedgelayer false)
+      (excludeedgelayer true)
       (linewidth 2.000000)
       (plotframeref false)
@@
       (drillshape 0)
       (scaleselection 1)
-      (outputdirectory ""))
+      (outputdirectory "Gerber bottom/"))
   )
   (net 0 "")
@@
   )
   (module MountingHole:MountingHole_2.2mm_M2_Pad (layer F.Cu)
-    (at 77.9018 178.5874)
-    (descr "Mounting Hole 2.2mm, M2")
-    (tags "mounting hole 2.2mm m2")
+    (at 79.4018 178.5874)
+    (descr "Mounting Hole 2.2mm, M2")
+    (tags "mounting hole 2.2mm m2")
